Commit message: Added new blocks

File: fetch_tufts/models/block/model1.urdf (robot description, URDF)
Before this commit: robot block, 1 links, 0 joints
Links:
- link block: mass 4.5 -> 0.01

File: fetch_tufts/models/block/model10.urdf (robot description, URDF)
Before this commit: robot block, 1 links, 0 joints
Links:
- link block: mass 0.25 -> 0.5625

File: fetch_tufts/models/block/model11.urdf (robot description, URDF)
Before this commit: robot block, 1 links, 0 joints
Links:
- link block: mass 0.1 -> 0.625

File: fetch_tufts/models/block/model12.urdf (robot description, URDF)
Before this commit: robot block, 1 links, 0 joints
Links:
- link block: mass 0.08 -> 0.6875

File: fetch_tufts/models/block/model13.urdf (robot description, URDF)
Before this commit: robot block, 1 links, 0 joints
Links:
- link block: mass 0.06 -> 0.75

File: fetch_tufts/models/block/model14.urdf (robot description, URDF)
Before this commit: robot block, 1 links, 0 joints
Links:
- link block: mass 0.04 -> 0.8125

File: fetch_tufts/models/block/model15.urdf (robot description, URDF)
Before this commit: robot block, 1 links, 0 joints
Links:
- link block: mass 0.02 -> 0.875

File: fetch_tufts/models/block/model17.urdf (robot description, URDF)
Before this commit: robot block, 1 links, 0 joints
Links:
- link block: mass 1.25 -> 1

File: fetch_tufts/models/block/model18.urdf (robot description, URDF)
Before this commit: robot block, 1 links, 0 joints
Links:
- link block: mass 0.75 -> 1.0625

File: fetch_tufts/models/block/model19.urdf (robot description, URDF)
Before this commit: robot block, 1 links, 0 joints
Links:
- link block: mass 0.9375 -> 1.125

File: fetch_tufts/models/block/model2.urdf (robot description, URDF)
Before this commit: robot block, 1 links, 0 joints
Links:
- link block: mass 4 -> 0.0625

File: fetch_tufts/models/block/model20.urdf (robot description, URDF)
Before this commit: robot block, 1 links, 0 joints
Links:
- link block: mass 0.9375 -> 1.1875

File: fetch_tufts/models/block/model21.urdf (robot description, URDF)
Before this commit: robot block, 1 links, 0 joints
Links:
- link block: mass 0.9375 -> 1.25

File: fetch_tufts/models/block/model22.urdf (robot description, URDF)
Before this commit: robot block, 1 links, 0 joints
Links:
- link block: mass 0.9375 -> 1.3125

File: fetch_tufts/models/block/model23.urdf (robot description, URDF)
Before this commit: robot block, 1 links, 0 joints
Links:
- link block: mass 0.9375 -> 1.375

File: fetch_tufts/models/block/model24.urdf (robot description, URDF)
Before this commit: robot block, 1 links, 0 joints
Links:
- link block: mass 0.9375 -> 1.4375

File: fetch_tufts/models/block/model25.urdf (robot description, URDF)
Before this commit: robot block, 1 links, 0 joints
Links:
- link block: mass 0.9375 -> 1.5

File: fetch_tufts/models/block/model3.urdf (robot description, URDF)
Before this commit: robot block, 1 links, 0 joints
Links:
- link block: mass 3.5 -> 0.125

File: fetch_tufts/models/block/model4.urdf (robot description, URDF)
Before this commit: robot block, 1 links, 0 joints
Links:
- link block: mass 3 -> 0.1875

File: fetch_tufts/models/block/model5.urdf (robot description, URDF)
Before this commit: robot block, 1 links, 0 joints
Links:
- link block: mass 2.5 -> 0.25
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